File: pocket/ver1.1/PCB/pocket.kicad_sch (KiCad schematic)
At the start: 60 parts, among them SW1 MX_SW_HS, SW10 MX_SW_HS, SW11 MX_SW_HS, SW12 MX_SW_HS, SW13 MX_SW_HS, SW14 MX_SW_HS, SW15 MX_SW_HS, SW16 MX_SW_HS, SW17 MX_SW_HS, SW18 MX_SW_HS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

Commit message: Add files via upload
Connections:
- net B2: now also SW10.1, SW20.1, SW29.1; no longer SW1.1, SW11.1, SW21.1
- net B3: now also SW12.1, SW2.1, SW22.1; no longer D1.1 (K), D10.1 (K), D2.1 (K), D3.1 (K), D4.1 (K), D5.1 (K), D6.1 (K), D7.1 (K), D8.1 (K), D9.1 (K)
- net B4: now also SW19.1, SW28.1, SW9.1; no longer SW17.1, SW26.1, SW7.1
- net B5: now also SW18.1, SW27.1, SW8.1; no longer SW16.1, SW6.1
- net C6: now also SW16.1, SW6.1; no longer SW10.1, SW20.1, SW29.1
- net D7: now also SW17.1, SW26.1, SW7.1; no longer SW19.1, SW28.1, SW9.1
- net E6: now also D21.1 (K), D22.1 (K), D23.1 (K), D24.1 (K), D25.1 (K), D26.1 (K), D27.1 (K), D28.1 (K), D29.1 (K); no longer SW18.1, SW27.1, SW8.1
- net F5: now also SW15.1, SW25.1, SW5.1; no longer SW14.1, SW24.1, SW4.1
- net F6: now also SW14.1, SW24.1, SW4.1; no longer SW15.1, SW25.1, SW5.1
- net B1: now reaches U1.16 (15/PB1)
- net B1: now also SW1.1, SW11.1, SW21.1
- net F7: now reaches U1.17 (A0/PF7)
- net F7: now also D1.1 (K), D10.1 (K), D2.1 (K), D3.1 (K), D4.1 (K), D5.1 (K), D6.1 (K), D7.1 (K), D8.1 (K), D9.1 (K)
- net D4: now reaches U1.7 (4/PD4)
- net D4: now also D11.1 (K), D12.1 (K), D13.1 (K), D14.1 (K), D15.1 (K), D16.1 (K), D17.1 (K), D18.1 (K), D19.1 (K), D20.1 (K)
- removed net B6: SW12.1, SW2.1, SW22.1, U1.13 (10/PB6)
- removed net D0: D21.1 (K), D22.1 (K), D23.1 (K), D24.1 (K), D25.1 (K), D26.1 (K), D27.1 (K), D28.1 (K), D29.1 (K), U1.6 (3/PD0)
- removed net D1: D11.1 (K), D12.1 (K), D13.1 (K), D14.1 (K), D15.1 (K), D16.1 (K), D17.1 (K), D18.1 (K), D19.1 (K), D20.1 (K), U1.5 (2/PD1)
